Commit message: code update upto SLAM

File: 10_ROS2/04_my_mobile/install/my_robot_description/share/my_robot_description/urdf/robot_core.xacro (robot description, xacro)
@@ -32,4 +32,5 @@
         <parent link="base_link"/>
         <child link="left_wheel"/>
+        <axis xyz="0 1 0"/>
         <origin xyz="0 ${wheel_separation/2} 0" rpy="0 0 0"/>
     </joint>
